File: tfg_adaptador/tfg_adaptador.kicad_pcb (KiCad board)
At the start: 2 copper layers, 100 x 75 mm, 13 parts, among them J2 Screw_Terminal_01x03, U2 THVD1400D

Commit message: ACTUALIZACION PCB
Parts:
- added C2: 100nf, Capacitor_SMD:C_0805_2012Metric, F.Cu at (127.0, 122.0)
- added D1: BZX384xxxx, Diode_SMD:D_SOD-323, F.Cu at (123.2, 109.5)
- added D2: BZX384xxxx, Diode_SMD:D_SOD-323, F.Cu at (123.2, 112.5)
- added D3: BZX384xxxx, Diode_SMD:D_SOD-323, F.Cu at (123.2, 115.5)
- added D4: BZX384xxxx, Diode_SMD:D_SOD-323, F.Cu at (123.2, 118.4)
- added IC1: TPS4H000AQPWPRQ1, freno:SOP65P640X120-20N, F.Cu at (116.5, 93.5)
- added J1: Screw_Terminal_01x08, terminal02x08:terminal02x08, F.Cu at (81.4, 106.5)
- added J3: Screw_Terminal_01x08, terminal02x08:terminal02x08, F.Cu at (81.3, 131.5)
- added J4: Screw_Terminal_01x08, terminal02x08:terminal02x08, F.Cu at (96.4, 131.5)
- added J5: Screw_Terminal_01x03, TerminalBlock_Phoenix:TerminalBlock_Phoenix_PT-1,5-3-5.0-H_1x03_P5.00mm_Horizontal, F.Cu at (106.0, 79.1)
- added R10: 3.3 K, Resistor_SMD:R_0805_2012Metric, F.Cu at (122.5, 136.9)
- added R11: 1K, Resistor_SMD:R_0805_2012Metric, F.Cu at (126.9, 128.1)
- added R12: 1K, Resistor_SMD:R_0805_2012Metric, F.Cu at (126.9, 131.0)
- added R13: 1K, Resistor_SMD:R_0805_2012Metric, F.Cu at (126.9, 133.9)
- added R14: 1K, Resistor_SMD:R_0805_2012Metric, F.Cu at (126.9, 136.9)
- added R4: 3.3 K, Resistor_SMD:R_0805_2012Metric, F.Cu at (118.1, 131.0)
- added R5: 1.7 K, Resistor_SMD:R_0805_2012Metric, F.Cu at (118.1, 133.9)
- added R6: 3.3 K, Resistor_SMD:R_0805_2012Metric, F.Cu at (118.1, 136.9)
- added R7: 1.7 K, Resistor_SMD:R_0805_2012Metric, F.Cu at (122.5, 128.1)
- added R8: 3.3 K, Resistor_SMD:R_0805_2012Metric, F.Cu at (122.5, 131.0)
- added R9: 1.7 K, Resistor_SMD:R_0805_2012Metric, F.Cu at (122.5, 133.9)
- added U2: MCP6001-OT, Package_TO_SOT_SMD:SOT-23-5, F.Cu at (118.5, 110.5)
- added U3: MCP6001-OT, Package_TO_SOT_SMD:SOT-23-5, F.Cu at (118.5, 115.1)
- added U4: MCP6001-OT, Package_TO_SOT_SMD:SOT-23-5, F.Cu at (118.5, 119.7)
- added U5: MCP6001-OT, Package_TO_SOT_SMD:SOT-23-5, F.Cu at (118.5, 124.3)
- C1: footprint Capacitor_THT:C_Disc_D3.0mm_W1.6mm_P2.50mm -> Capacitor_SMD:C_0805_2012Metric
- J2: value Screw_Terminal_01x03 -> Screw_Terminal_01x08; footprint TerminalBlock_Phoenix:TerminalBlock_Phoenix_PT-1,5-3-3.5-H_1x03_P3.50mm_Horizontal -> terminal02x08:terminal02x08
- R1: value 120 -> 10K; footprint Resistor_THT:R_Axial_DIN0207_L6.3mm_D2.5mm_P7.62mm_Horizontal -> Resistor_SMD:R_0805_2012Metric
- R2: value 4.7K -> 10K; footprint Resistor_THT:R_Axial_DIN0207_L6.3mm_D2.5mm_P7.62mm_Horizontal -> Resistor_SMD:R_0805_2012Metric
- R3: value 4.7K -> 1.7 K; footprint Resistor_THT:R_Axial_DIN0207_L6.3mm_D2.5mm_P7.62mm_Horizontal -> Resistor_SMD:R_0805_2012Metric
- moved R1 43.8 mm to (127.5, 118.5)
- moved R3 43.4 mm to (118.1, 128.1)
- moved J2 41.9 mm to (96.5, 106.5), turned to 90 degrees
- moved C1 38.9 mm to (127.0, 124.5)
- moved R2 38.4 mm to (127.5, 116.0)
- moved H1 21.5 mm to (83.5, 80.0)
- moved H2 21.5 mm to (83.5, 145.0)
- moved U1 18.6 mm to (119.0, 79.9)
- renumbered U2 to U1
Connections:
- net Net-(A1-GPIO0) renamed /SDA1
- net Net-(A1-GPIO1) renamed /SCL1
- net Net-(A1-GPIO2) renamed /SDA2
- net Net-(A1-GPIO3) renamed /SCL2
- A1 pad 10: unconnected-(A1-GPIO7-Pad10) -> /DOUT4
- A1 pad 11: unconnected-(A1-GPIO8-Pad11) -> /SIN1
- A1 pad 12: unconnected-(A1-GPIO9-Pad12) -> /SIN2
- A1 pad 14: unconnected-(A1-GPIO10-Pad14) -> /SIN3
- A1 pad 15: unconnected-(A1-GPIO11-Pad15) -> /SIN4
- A1 pad 17: Net-(A1-GPIO13) -> +3.3V
- A1 pad 20: Net-(A1-GPIO15) -> Net-(A1-GPIO14)
- A1 pad 21: unconnected-(A1-GPIO16-Pad21) -> /AOUT1
- A1 pad 22: unconnected-(A1-GPIO17-Pad22) -> /AOUT2
- A1 pad 24: unconnected-(A1-GPIO18-Pad24) -> /AOUT3
- A1 pad 25: unconnected-(A1-GPIO19-Pad25) -> /AOUT4
- A1 pad 40: unconnected-(A1-VBUS-Pad40) -> +5V
- A1 pad 6: unconnected-(A1-GPIO4-Pad6) -> /DOUT1
- A1 pad 7: unconnected-(A1-GPIO5-Pad7) -> /DOUT2
- A1 pad 9: unconnected-(A1-GPIO6-Pad9) -> /DOUT3
- R1 pad 1: Net-(J2-Pin_2) -> GND
- R1 pad 2: Net-(J2-Pin_1) -> Net-(A1-GPIO14)
- R2 pad 1: GND -> +3.3V
- R2 pad 2: Net-(J2-Pin_2) -> +3.3V
- R3 pad 1: Net-(J2-Pin_1) -> Net-(U2--)
- R3 pad 2: GND -> /AOUT1
- U1 pad 1: Net-(A1-GPIO13) -> +3.3V
- U1 pad 4: Net-(A1-GPIO15) -> Net-(A1-GPIO14)
- U1 pad 6: Net-(J2-Pin_1) -> Net-(J5-Pin_1)
- U1 pad 7: Net-(J2-Pin_2) -> Net-(J5-Pin_2)
Routing:
- net +3.3V: track 99.0 -> 0.00 mm
- net Net-(J2-Pin_2): track 87.6 -> 0.00 mm
- net Net-(J2-Pin_1): track 54.2 -> 0.00 mm
- net Net-(A1-GPIO13): track 48.0 -> 0.00 mm
- net /SDA2: track 43.9 -> 0.00 mm
- net /SCL2: track 36.0 -> 0.00 mm
- net Net-(A1-GPIO14): track 34.4 -> 0.00 mm
- net Net-(A1-GPIO15): track 29.9 -> 0.00 mm
- net /SDA1: track 29.8 -> 0.00 mm
- net /SCL1: track 21.8 -> 0.00 mm
Other:
- board size 100 x 75 mm -> 123 x 75 mm
