File: tfg_adaptador/tfg_adaptador.kicad_sch (KiCad schematic)
At the start: 13 parts, among them J2 Screw_Terminal_01x03, U2 THVD1400D

Commit message: ACTUALIZACION PCB
Parts:
- removed J2: Screw_Terminal_01x03, TerminalBlock_Phoenix:TerminalBlock_Phoenix_PT-1,5-3-3.5-H_1x03_P3.50mm_Horizontal, symbol Connector:Screw_Terminal_01x03
- added C2: 100nf, Capacitor_SMD:C_0805_2012Metric, symbol Device:C
- added D1, D2, D3, D4: BZX384xxxx, Diode_SMD:D_SOD-323, symbol Diode:BZX384xxxx
- added IC1: TPS4H000AQPWPRQ1, freno:SOP65P640X120-20N, symbol TPS4H000AQPWPRQ1:TPS4H000AQPWPRQ1
- added J1, J2, J3, J4: Screw_Terminal_01x08, terminal02x08:terminal02x08, symbol Connector:Screw_Terminal_01x08
- added J5: Screw_Terminal_01x03, TerminalBlock_Phoenix:TerminalBlock_Phoenix_PT-1,5-3-5.0-H_1x03_P5.00mm_Horizontal, symbol Connector:Screw_Terminal_01x03
- added R10, R4, R6, R8: 3.3 K, Resistor_SMD:R_0805_2012Metric, symbol Device:R
- added R11, R12, R13, R14: 1K, Resistor_SMD:R_0805_2012Metric, symbol Device:R
- added R5, R7, R9: 1.7 K, Resistor_SMD:R_0805_2012Metric, symbol Device:R
- added U2, U3, U4, U5: MCP6001-OT, Package_TO_SOT_SMD:SOT-23-5, symbol Amplifier_Operational:MCP6001-OT
- C1: footprint Capacitor_THT:C_Disc_D3.0mm_W1.6mm_P2.50mm -> Capacitor_SMD:C_0805_2012Metric
- R1: value 120 -> 10K; footprint Resistor_THT:R_Axial_DIN0207_L6.3mm_D2.5mm_P7.62mm_Horizontal -> Resistor_SMD:R_0805_2012Metric
- R2: value 4.7K -> 10K; footprint Resistor_THT:R_Axial_DIN0207_L6.3mm_D2.5mm_P7.62mm_Horizontal -> Resistor_SMD:R_0805_2012Metric
- R3: value 4.7K -> 1.7 K; footprint Resistor_THT:R_Axial_DIN0207_L6.3mm_D2.5mm_P7.62mm_Horizontal -> Resistor_SMD:R_0805_2012Metric
- renumbered U2 to U1
Connections:
- net +3.3V: now also A1.17 (GPIO13), R2.1, R2.2, U1.1 (RO), C2.2
- net GND: now also R1.1, C2.1, D1.2 (A), D2.2 (A), D3.2 (A), D4.2 (A), IC1.10 (GND), J5.3 (Pin_3), R10.2, R4.2, R6.2, R8.2; no longer R2.1, R3.2
- net SCL1: now reaches A1.2 (GPIO1), MD1.13 (SCL)
- net SDA1: now reaches A1.1 (GPIO0), MD1.14 (SDA)
- net at A1.19 (GPIO14), U1.2 (~{RE}), U1.3 (DE): now also A1.20 (GPIO15), R1.2, U1.4 (DI)
- net DOUT4: now reaches A1.10 (GPIO7)
- net DOUT4: now also D4.1 (K), R14.2
- net SIN1: now reaches A1.11 (GPIO8)
- net SIN1: now also IC1.1 (IN1)
- net SIN2: now reaches A1.12 (GPIO9)
- net SIN2: now also IC1.2 (IN2)
- net SIN3: now reaches A1.14 (GPIO10)
- net SIN3: now also IC1.3 (IN3)
- net SIN4: now reaches A1.15 (GPIO11)
- net SIN4: now also IC1.4 (IN4)
- net AOUT1: now reaches A1.21 (GPIO16)
- net AOUT1: now also R3.2, R4.1
- net AOUT2: now reaches A1.22 (GPIO17)
- net AOUT2: now also R5.2, R6.1
- net AOUT3: now reaches A1.24 (GPIO18)
- net AOUT3: now also R7.2, R8.1
- net AOUT4: now reaches A1.25 (GPIO19)
- net AOUT4: now also R10.1, R9.2
- net SDA2: now reaches A1.4 (GPIO2), MD2.14 (SDA)
- net +5V: now reaches A1.40 (VBUS)
- net +5V: now also IC1.17 (VS_1)
- net SCL2: now reaches A1.5 (GPIO3), MD2.13 (SCL)
- net DOUT1: now reaches A1.6 (GPIO4)
- net DOUT1: now also D1.1 (K), R11.2
- net DOUT2: now reaches A1.7 (GPIO5)
- net DOUT2: now also D2.1 (K), R12.2
- net DOUT3: now reaches A1.9 (GPIO6)
- net DOUT3: now also D3.1 (K), R13.2
- new net: R9.1, U5.1, U5.4 (-)
- new net: J5.1 (Pin_1), U1.6 (A)
- new net: J5.2 (Pin_2), U1.7 (B)
- new net: R3.1, U2.1, U2.4 (-)
- new net: R5.1, U3.1, U3.4 (-)
- new net: R7.1, U4.1, U4.4 (-)
- new net AIN1: J2.8 (Pin_8), U2.3 (+)
- new net AIN2: J2.7 (Pin_7), U3.3 (+)
- new net AIN3: J2.6 (Pin_6), U4.3 (+)
- new net AIN4: J2.5 (Pin_5), U5.3 (+)
- new net DI1: J2.1 (Pin_1), R11.1
- new net DI2: J2.2 (Pin_2), R12.1
- new net DI3: J2.3 (Pin_3), R13.1
- new net DI4: J2.4 (Pin_4), R14.1
- new net SOUT1: IC1.20 (OUT1), J4.8 (Pin_8)
- new net SOUT2: IC1.19 (OUT2), J4.7 (Pin_7)
- new net SOUT3: IC1.16 (OUT3), J4.6 (Pin_6)
- new net SOUT4: IC1.15 (OUT4), J4.5 (Pin_5)
Other:
- note added: "485 ADAPTER"
- note added: "ANALOGIC INPUTS"
- note added: "DIGITAL INPUTS"
- note added: "DIGITAL OUTPUTS"
- note added: "LOADCELL 1"
- note added: "LOADCELL 2"
- note added: "RASPBERRY PICO"
- moved on the sheet: A1, C1, H1, H2, H3, H4, MD1, MD2, U1
